Commit message: ダッキーのurdfを追加

File: urdf/drones/legacy/iris.xacro (robot description, xacro)
@@ -10,5 +10,5 @@
   <xacro:property name="body_length" value="0.18" /> <!-- [m] 0.10 -->
   <xacro:property name="body_width" value="0.12" /> <!-- [m] 0.10 -->
-  <xacro:property name="body_height" value="0.10" /> <!-- [m] -->
+  <xacro:property name="body_height" value="0.15" /> <!-- [m] -->
   <xacro:property name="mass_rotor" value="0.005" /> <!-- [kg] -->
   <xacro:property name="arm_length_front_x" value="0.1422" /> <!-- [m] 0.1425  0.22 -->
@@ -28,5 +28,5 @@
   <xacro:property name="rotor_drag_coefficient" value="8.06428e-05" />
   <xacro:property name="rolling_moment_coefficient" value="0.000001" />
-  <xacro:property name="color" value="DarkGrey" />
+  <xacro:property name="color" value="White" />
   <!-- Property Blocks -->
   <xacro:property name="body_inertia">
@@ -42,5 +42,4 @@
   </xacro:property>
   <!-- Included URDF Files -->
-  <!-- <xacro:include filename="$(find rotors_description)/urdf/multirotor_base.xacro" /> -->
   <xacro:include filename="$(find agri_resources)/urdf/drones/multirotor_base.xacro" />
   <!-- Instantiate multirotor_base_macro once -->
@@ -58,150 +57,11 @@
   </xacro:multirotor_base_macro>
   <xacro:property name="M_PI" value="3.1415926535897931" />
-  <!-- Recorder cameras -->
-  <xacro:include filename="$(find agri_resources)/urdf/sensors/recorder_camera.xacro" />
-  <!--
-<xacro:recorder_camera
-    name="recorder_cam_front_with_uav"
-    parent="base_link"
-    ros_topic="recorder_cam_front_with_uav"
-    update_rate="90"
-    res_x="1680"
-    res_y="1050"
-    image_format="R8G8B8"
-    hfov="81"
-    video_dir="/home/aurelien/Videos/shots/"
-    video_filename="cam_front_with_uav"
-    video_fileext="avi">
-    <origin xyz="-0.8 0.0 0.12" rpy="0 0 0"/>
-  </xacro:recorder_camera>
--->
-  <!--
-  <xacro:recorder_camera
-    name="recorder_cam_front_with_uav2"
-    parent="base_link"
-    ros_topic="recorder_cam_front_with_uav2"
-    update_rate="30"
-    res_x="1680"
-    res_y="1050"
-    image_format="R8G8B8"
-    hfov="81"
-    video_dir="/home/aurelien/Videos/shots/"
-    video_filename="cam_front_with_uav2"
-    video_fileext="avi">
-    <origin xyz="-0.3 0.0 0.15" rpy="0 0.2 0"/>
-  </xacro:recorder_camera>
-  -->
-  <!--
-  <xacro:recorder_camera
-    name="recorder_cam_rear_with_uav"
-    parent="base_link"
-    ros_topic="recorder_cam_rear_with_uav"
-    update_rate="30"
-    res_x="1680"
-    res_y="1050"
-    image_format="R8G8B8"
-    hfov="81"
-    video_dir="/home/aurelien/Videos/shots/"
-    video_filename="cam_rear_with_uav"
-    video_fileext="avi">
-    <origin xyz="0.6 0.0 -0.12" rpy="0 ${-20*M_PI/180} ${180*M_PI/180}"/>
-  </xacro:recorder_camera>
-  -->
-  <!--
-  <xacro:recorder_camera
-    name="recorder_cam_rear_with_uav2"
-    parent="base_link"
-    ros_topic="recorder_cam_rear_with_uav2"
-    update_rate="90"
-    res_x="1680"
-    res_y="1050"
-    image_format="R8G8B8"
-    hfov="81"
-    video_dir="/home/aurelien/Videos/shots/"
-    video_filename="cam_rear_with_uav2"
-    video_fileext="avi">
-    <origin xyz="0.4 0.0 0.12" rpy="0 ${20*M_PI/180} ${180*M_PI/180}"/>
-  </xacro:recorder_camera>
-  -->
-  <!-- Recorder cameras END -->
-  <!-- Sonar height sensor -->
-  <xacro:include filename="$(find agri_resources)/urdf/sensors/sonar_sensor.urdf.xacro" />
- <!--
-  <xacro:sonar_sensor
-    name="sonar"
-    parent="base_link"
-    ros_topic="sonar_down"
-    update_rate="10"
-    min_range="0.01"
-    max_range="50.0"
-    field_of_view="${1*M_PI/180}"
-    ray_count="1"
-    sensor_mesh="lidar_lite_v2/meshes/lidar_lite_v2.dae">
-    <origin xyz="0.12 0.0 0.0" rpy="0 ${90*M_PI/180} 0"/>
-  </xacro:sonar_sensor>
-     -->
-    <!-- Frontal range sensor -->
- <!--  <xacro:sonar_sensor
-    name="sonar2"
-    parent="base_link"
-    ros_topic="sonar_front"
-    update_rate="10"
-    min_range="0.01"
-    max_range="50.0"
-    field_of_view="${1*M_PI/180}"
-    ray_count="1"
-    sensor_mesh="lidar_lite_v2_withRay/meshes/lidar_lite_v2_withRay.dae">
-    <origin xyz="0.13 0.0 0.02" rpy="0 0 0"/>
-  </xacro:sonar_sensor>
--->
-<!--
-  <xacro:include filename="$(find ego_planner)/../../urdf/sensors/lidar_sensor.urdf.xacro" />
-   <xacro:lidar_sensor
-    name="sonar2"
-    parent="base_link"
-    ros_topic="sonar_front"
-    update_rate="10"
-    min_range="0.01"
-    max_range="10.0"
-    field_of_view_horizontal="${70*M_PI/180}"
-    field_of_view_vertical="${1*M_PI/180}"
-    ray_count_horizontal="140"
-    ray_count_vertical="1"
-    sensor_mesh="lidar_lite_v2_withRay/meshes/lidar_lite_v2_withRay.dae">
-    <origin xyz="0.13 0.0 0.02" rpy="0 0 0"/>
-  </xacro:lidar_sensor>
--->
-  <!-- Downward facing camera -->
-  <xacro:include filename="$(find agri_resources)/urdf/sensors/generic_camera.urdf.xacro" />
-  <xacro:generic_camera
-    name="iris/bottom"
-    parent="base_link"
-    ros_topic="image_raw"
-    cam_info_topic="camera_info"
-    update_rate="60"
-    res_x="640"
-    res_y="360"
-    image_format="R8G8B8"
-    hfov="81"
-    framename="iris_bottomcam">
-    <origin xyz="0.14 0.0 -0.02" rpy="0 ${M_PI/2} 0"/>
-  </xacro:generic_camera>
-  <!-- Front facing camera -->
-  <xacro:include filename="$(find agri_resources)/urdf/sensors/generic_camera.urdf.xacro" />
-  <xacro:generic_camera
-    name="iris/front"
-    parent="base_link"
-    ros_topic="image_front_raw"
-    cam_info_topic="camera_front_info"
-    update_rate="25"
-    res_x="640"
-    res_y="360"
-    image_format="R8G8B8"
-    hfov="81"
-    framename="iris_frontcam">
-    <origin xyz="0.17 0.0 0.0" rpy="0 0 0"/>
-  </xacro:generic_camera>
+  <!-- Realsense -->
+  <xacro:include filename="$(find agri_resources)/urdf/sensors/d435/_d435.urdf.xacro" />
+  <xacro:sensor_d435 name="camera" topics_ns="camera" parent="base_link" publish_pointcloud="true">
+    <origin xyz="0.1 0 0.19" rpy="0 0 0" />
+  </xacro:sensor_d435>
   <!-- Instantiate rotors -->
-  <xacro:vertical_rotor
+  <!-- <xacro:vertical_rotor
     robot_namespace="${namespace}"
     suffix="front_right"
@@ -284,4 +144,4 @@
     <origin xyz="-${arm_length_back_x} -${arm_length_back_y} ${rotor_offset_top}" rpy="0 0 0" />
     <xacro:insert_block name="rotor_inertia" />
-  </xacro:vertical_rotor>
+  </xacro:vertical_rotor> -->
 </robot>

File: urdf/drones/legacy/iris_base.xacro (robot description, xacro)
@@ -1,139 +1,103 @@
 <?xml version="1.0"?>
-<robot name="iris" xmlns:xacro="http://ros.org/wiki/xacro">
-  <xacro:include filename="$(find rotors_description)/urdf/component_snippets.xacro" />
-  <!-- Instantiate iris "mechanics" -->
-  <xacro:include filename="$(find agri_resources)/urdf/drones/iris.xacro" />
-  <!-- Specify reference parameters for GNSS receiver. -->
-  <xacro:include filename="$(find agri_resources)/urdf/drones/gps_home_location.xacro" />
-  <!-- Reference heading is equivalent to rotating Gazebo's map.
-       We do not use it for we would loose the match X=North, Y=West -->
-  <!-- in degrees, 0 so North is towards positive X values, and East is towards negative Y values -->
-  <xacro:property name="referenceHeading" value="0" />
-  <!-- Instantiate a controller. -->
-  <xacro:controller_plugin_macro
-    namespace="${namespace}"
-    imu_sub_topic="imu"
-    >
-  </xacro:controller_plugin_macro>
-  <!-- Mount an ADIS16448 IMU. -->
-  <xacro:imu_plugin_macro
-    namespace="${namespace}"
-    imu_suffix=""
-    parent_link="base_link"
-    imu_topic="imu"
-    mass_imu_sensor="0.015"
-    gyroscope_noise_density="0.0003394"
-    gyroscopoe_random_walk="0.000038785"
-    gyroscope_bias_correlation_time="1000.0"
-    gyroscope_turn_on_bias_sigma="0.0087"
-    accelerometer_noise_density="0.004"
-    accelerometer_random_walk="0.006"
-    accelerometer_bias_correlation_time="300.0"
-    accelerometer_turn_on_bias_sigma="0.1960"
-  >
-    <inertia ixx="0.00001" ixy="0.0" ixz="0.0" iyy="0.00001" iyz="0.0" izz="0.00001" />
-    <origin xyz="0 0 0" rpy="0 0 0" />
-  </xacro:imu_plugin_macro>
-  <!-- Mount a GNSS receiver. -->
-  <gazebo>
-    <plugin name="${namespace}_gps_sim" filename="libhector_gazebo_ros_gps.so">
-      <alwaysOn>true</alwaysOn>
-      <topicName>${namespace}/fix</topicName>
-      <velocityTopicName>${namespace}/fix_velocity</velocityTopicName>
-      <referenceLatitude>${referenceLatitude}</referenceLatitude>
-      <referenceLongitude>${referenceLongitude}</referenceLongitude>
-      <referenceHeading>${referenceHeading}</referenceHeading>
-      <referenceAltitude>${referenceAltitude}</referenceAltitude>
-      <!-- Sensor errors model for GPS Position measures -->
-      <!-- Units: [m], and [1/s] for drift frequency -->
-      <!-- For now, use Ardupilot's internal error models -->
-      <offset>0 0 0</offset>
-      <drift>0 0 0</drift>
-      <driftFrequency>0 0 0</driftFrequency>
-      <gaussianNoise>0 0 0</gaussianNoise>
-      <scaleError>1 1 1</scaleError>
-      <!-- Note:
-       For the moment there is no barometer, so axis Z of the GPS is
-       used as a barometer sensor (with the according error model) -->
-      <!-- Sensor errors model for GPS Velocity measures -->
-      <!-- Units: [m/s], and [1/s] for drift frequency -->
-      <!-- For now, use Ardupilot's internal error models -->
-      <velocityOffset>0 0 0</velocityOffset>
-      <velocityDrift>0 0 0</velocityDrift>
-      <velocityDriftFrequency>0 0 0</velocityDriftFrequency>
-      <velocityGaussianNoise>0 0 0</velocityGaussianNoise>
-      <velocityScaleError>1 1 1</velocityScaleError>
-      <!-- Note:
-        The velocity Z does not really make sense, it is not used by
-        Ardupilot (right?).
-        However Z velocity drift is added to the Z position drift. -->
-      <!-- Explanations:
-         offset:          constant added to the real value
-         gaussian noise:  randomly generated noise added to the real value
-         drift:           amount of drift
-         drift frequency: time constant (as a frequency) for the drift
-         scale error:     scaling of the real value (before adding other noises)
-       -->
-    </plugin>
-  </gazebo>
-  <xacro:if value="$(arg enable_ground_truth)">
-    <!-- Mount an IMU providing ground truth. -->
-    <xacro:imu_plugin_macro
-      namespace="${namespace}"
-      imu_suffix="gt"
-      parent_link="base_link"
-      imu_topic="ground_truth/imu"
-      mass_imu_sensor="0.00001"
-      gyroscope_noise_density="0.0"
-      gyroscopoe_random_walk="0.0"
-      gyroscope_bias_correlation_time="1000.0"
-      gyroscope_turn_on_bias_sigma="0.0"
-      accelerometer_noise_density="0.0"
-      accelerometer_random_walk="0.0"
-      accelerometer_bias_correlation_time="300.0"
-      accelerometer_turn_on_bias_sigma="0.0"
-    >
-      <inertia ixx="0.00001" ixy="0.0" ixz="0.0" iyy="0.00001" iyz="0.0" izz="0.00001" />
-      <origin xyz="0 0 0" rpy="0 0 0" />
-    </xacro:imu_plugin_macro>
-    <!-- Mount a generic odometry sensor providing ground truth. -->
-    <xacro:odometry_plugin_macro
-      namespace="${namespace}/ground_truth"
-      odometry_sensor_suffix="gt"
-      parent_link="base_link"
-      pose_topic="pose"
-      pose_with_covariance_topic="pose_with_covariance"
-      position_topic="position"
-      transform_topic="transform"
-      odometry_topic="odometry"
-      parent_frame_id="world"
-      mass_odometry_sensor="0.00001"
-      measurement_divisor="1"
-      measurement_delay="0"
-      unknown_delay="0.0"
-      noise_normal_position="0 0 0"
-      noise_normal_quaternion="0 0 0"
-      noise_normal_linear_velocity="0 0 0"
-      noise_normal_angular_velocity="0 0 0"
-      noise_uniform_position="0 0 0"
-      noise_uniform_quaternion="0 0 0"
-      noise_uniform_linear_velocity="0 0 0"
-      noise_uniform_angular_velocity="0 0 0"
-      enable_odometry_map="false"
-      odometry_map=""
-      image_scale=""
-    >
-      <inertia ixx="0.00001" ixy="0.0" ixz="0.0" iyy="0.00001" iyz="0.0" izz="0.00001" /> <!-- [kg.m^2] [kg.m^2] [kg.m^2] [kg.m^2] [kg.m^2] [kg.m^2] -->
-      <origin xyz="0.0 0.0 0.0" rpy="0.0 0.0 0.0" />
-    </xacro:odometry_plugin_macro>
-  </xacro:if>
-  <xacro:if value="$(arg enable_logging)">
-    <!-- Instantiate a logger -->
-    <xacro:bag_plugin_macro
-      namespace="${namespace}"
-      bag_file="$(arg log_file)"
-      rotor_velocity_slowdown_sim="${rotor_velocity_slowdown_sim}"
-    >
-    </xacro:bag_plugin_macro>
-  </xacro:if>
+<robot xmlns:xacro="http://ros.org/wiki/xacro" name="iris_demo">
+  <xacro:include filename="$(find agri_resources)/urdf/drones/iris.xacro"/>
+  <!-- Define a macro for the LiftDrag plugin -->
+  <xacro:macro name="lift_drag_plugin" params="name a0 alpha_stall cla cda cma cla_stall cda_stall cma_stall area air_density cp forward upward link_name">
+    <gazebo reference="${link_name}">
+      <plugin name="${name}" filename="libLiftDragPlugin.so">
+        <a0>${a0}</a0>
+        <alpha_stall>${alpha_stall}</alpha_stall>
+        <cla>${cla}</cla>
+        <cda>${cda}</cda>
+        <cma>${cma}</cma>
+        <cla_stall>${cla_stall}</cla_stall>
+        <cda_stall>${cda_stall}</cda_stall>
+        <cma_stall>${cma_stall}</cma_stall>
+        <area>${area}</area>
+        <air_density>${air_density}</air_density>
+        <cp>${cp}</cp>
+        <forward>${forward}</forward>
+        <upward>${upward}</upward>
+      </plugin>
+    </gazebo>
+  </xacro:macro>
+  <!-- Instantiate the LiftDrag plugin macros for all rotor blades -->
+  <xacro:lift_drag_plugin name="rotor_0_blade_1" a0="0.3" alpha_stall="1.4" cla="4.2500" cda="0.10" cma="0.00" cla_stall="-0.025" cda_stall="0.0" cma_stall="0.0" area="0.002" air_density="1.2041" cp="0.084 0 0" forward="0 1 0" upward="0 0 1" link_name="rotor_0"/>
+  <xacro:lift_drag_plugin name="rotor_0_blade_2" a0="0.3" alpha_stall="1.4" cla="4.2500" cda="0.10" cma="0.00" cla_stall="-0.025" cda_stall="0.0" cma_stall="0.0" area="0.002" air_density="1.2041" cp="-0.084 0 0" forward="0 -1 0" upward="0 0 1" link_name="rotor_0"/>
+  <xacro:lift_drag_plugin name="rotor_1_blade_1" a0="0.3" alpha_stall="1.4" cla="4.2500" cda="0.10" cma="0.00" cla_stall="-0.025" cda_stall="0.0" cma_stall="0.0" area="0.002" air_density="1.2041" cp="0.084 0 0" forward="0 1 0" upward="0 0 1" link_name="rotor_1"/>
+  <xacro:lift_drag_plugin name="rotor_1_blade_2" a0="0.3" alpha_stall="1.4" cla="4.2500" cda="0.10" cma="0.00" cla_stall="-0.025" cda_stall="0.0" cma_stall="0.0" area="0.002" air_density="1.2041" cp="-0.084 0 0" forward="0 -1 0" upward="0 0 1" link_name="rotor_1"/>
+  <xacro:lift_drag_plugin name="rotor_2_blade_1" a0="0.3" alpha_stall="1.4" cla="4.2500" cda="0.10" cma="0.00" cla_stall="-0.025" cda_stall="0.0" cma_stall="0.0" area="0.002" air_density="1.2041" cp="0.084 0 0" forward="0 -1 0" upward="0 0 1" link_name="rotor_2"/>
+  <xacro:lift_drag_plugin name="rotor_2_blade_2" a0="0.3" alpha_stall="1.4" cla="4.2500" cda="0.10" cma="0.00" cla_stall="-0.025" cda_stall="0.0" cma_stall="0.0" area="0.002" air_density="1.2041" cp="-0.084 0 0" forward="0 1 0" upward="0 0 1" link_name="rotor_2"/>
+  <xacro:lift_drag_plugin name="rotor_3_blade_1" a0="0.3" alpha_stall="1.4" cla="4.2500" cda="0.10" cma="0.00" cla_stall="-0.025" cda_stall="0.0" cma_stall="0.0" area="0.002" air_density="1.2041" cp="0.084 0 0" forward="0 -1 0" upward="0 0 1" link_name="rotor_3"/>
+  <xacro:lift_drag_plugin name="rotor_3_blade_2" a0="0.3" alpha_stall="1.4" cla="4.2500" cda="0.10" cma="0.00" cla_stall="-0.025" cda_stall="0.0" cma_stall="0.0" area="0.002" air_density="1.2041" cp="-0.084 0 0" forward="0 1 0" upward="0 0 1" link_name="rotor_3"/>
+  <xacro:macro name="arducopter_plugin" params="">
+    <gazebo>
+      <plugin name="arducopter_plugin" filename="libArduPilotPlugin.so">
+        <fdm_addr>127.0.0.1</fdm_addr>
+        <fdm_port_in>9002</fdm_port_in>
+        <fdm_port_out>9003</fdm_port_out>
+        <modelXYZToAirplaneXForwardZDown>0 0 0 3.141593 0 0</modelXYZToAirplaneXForwardZDown>
+        <gazeboXYZToNED>0 0 0 3.141593 0 0</gazeboXYZToNED>
+        <imuName>iris::iris/imu_link::imu_sensor</imuName>
+        <connectionTimeoutMaxCount>5</connectionTimeoutMaxCount>
+        <control channel="0">
+          <type>VELOCITY</type>
+          <offset>0</offset>
+          <p_gain>0.20</p_gain>
+          <i_gain>0</i_gain>
+          <d_gain>0</d_gain>
+          <i_max>0</i_max>
+          <i_min>0</i_min>
+          <cmd_max>2.5</cmd_max>
+          <cmd_min>-2.5</cmd_min>
+          <jointName>rotor_0_joint</jointName>
+          <multiplier>838</multiplier>
+          <controlVelocitySlowdownSim>1</controlVelocitySlowdownSim>
+        </control>
+        <control channel="1">
+          <type>VELOCITY</type>
+          <offset>0</offset>
+          <p_gain>0.20</p_gain>
+          <i_gain>0</i_gain>
+          <d_gain>0</d_gain>
+          <i_max>0</i_max>
+          <i_min>0</i_min>
+          <cmd_max>2.5</cmd_max>
+          <cmd_min>-2.5</cmd_min>
+          <jointName>rotor_1_joint</jointName>
+          <multiplier>838</multiplier>
+          <controlVelocitySlowdownSim>1</controlVelocitySlowdownSim>
+        </control>
+        <control channel="2">
+          <type>VELOCITY</type>
+          <offset>0</offset>
+          <p_gain>0.20</p_gain>
+          <i_gain>0</i_gain>
+          <d_gain>0</d_gain>
+          <i_max>0</i_max>
+          <i_min>0</i_min>
+          <cmd_max>2.5</cmd_max>
+          <cmd_min>-2.5</cmd_min>
+          <jointName>rotor_2_joint</jointName>
+          <multiplier>-838</multiplier>
+          <controlVelocitySlowdownSim>1</controlVelocitySlowdownSim>
+        </control>
+        <control channel="3">
+          <type>VELOCITY</type>
+          <offset>0</offset>
+          <p_gain>0.20</p_gain>
+          <i_gain>0</i_gain>
+          <d_gain>0</d_gain>
+          <i_max>0</i_max>
+          <i_min>0</i_min>
+          <cmd_max>2.5</cmd_max>
+          <cmd_min>-2.5</cmd_min>
+          <jointName>rotor_3_joint</jointName>
+          <multiplier>-838</multiplier>
+          <controlVelocitySlowdownSim>1</controlVelocitySlowdownSim>
+        </control>
+      </plugin>
+    </gazebo>
+  </xacro:macro>
+  <xacro:arducopter_plugin/>
 </robot>
