Commit message: add realsense config file

File: urdf/drones/duckey.urdf (robot description, URDF)
Before this commit: robot duckey_drone, 1 links, 0 joints
Links:
- removed link base_link
- added link imu; visual mesh filename=package://agri_resources/meshes/drones/duckey.dae

Commit message: edit config file

File: urdf/drones/duckey.urdf (robot description, URDF)
Before this commit: robot duckey_drone, 1 links, 0 joints
Links:
- added link camera_link
Joints:
- added joint imu_to_camera: type fixed, parent imu, child camera_link, origin xyz=-0.015 0.03 0.035 rpy=1.57 -1.57 0

Commit message: rotate fix

File: urdf/drones/duckey.urdf (robot description, URDF)
Before this commit: robot duckey_drone, 2 links, 1 joints
Joints:
- joint imu_to_camera: origin xyz=-0.015 0.03 0.035 rpy=1.57 -1.57 0 -> xyz=-0.015 0.03 0.035 rpy=3.14 0 0

Commit message: debug

File: urdf/drones/duckey.urdf (robot description, URDF)
Before this commit: robot duckey_drone, 2 links, 1 joints
Joints:
- joint imu_to_camera: origin xyz=-0.015 0.03 0.035 rpy=3.14 0 0 -> xyz=0.03 -0.025 0.035 rpy=3.14 0 0

Commit message: add network script

File: urdf/drones/duckey.urdf (robot description, URDF)
Before this commit: robot duckey_drone, 2 links, 1 joints
Links:
- removed link imu
- added link base_link; visual mesh filename=package://agri_resources/meshes/drones/duckey.dae
Joints:
- joint imu_to_camera: parent imu -> base_link
